File: effectiveRangeHat_simple.kicad_pcb (KiCad board)
At the start: 8 copper layers, 30.6 x 66.8 mm, 124 parts, among them J1 Raspberry_Pi_2_3, J10 Conn_02x08_Odd_Even, J11 Conn_01x08, J2 BATT_CON, J3 PWR_HDR, J4 NCT_BYPASS, J5 PeriHDR, J8 I2C_EXT, P1 USB4105GFA120, Q1 2N7002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

Commit message: Bumping release from 1.9.0 to 1.10.0
Other:
- board text added: "MrHat v1.10.0"
- board text removed: "MrHat v1.9.0"
Changed lines of the file:
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@@
 	(title_block
 		(title "Effective Range: MrHat")
-		(date "2024-04-19")
-		(rev "1.9.0")
+		(date "2024-06-17")
+		(rev "1.10.0")
 		(company "Effective Range Kft.")
 		(comment 1 "visit https://creativecommons.org/licenses/by/4.0/")
@@
 		(layer "F.SilkS")
 	)
-	(gr_text "MrHat v1.9.0"
+	(gr_text "MrHat v1.10.0"
 		(at 108.2802 96.4692 90)
 		(layer "B.Cu")
