File: ChargeEnableLogic.kicad_sch (KiCad schematic)
At the start: 29 parts, among them U3 PIC18F16Q20, U4 RX8130CE, U7 SN74CBTLV3257RSVR, U9 GSF7002DW

Commit message: fix: erc errors
Changed lines of the file:
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@@
 	)
 	(junction
+		(at 229.87 86.36)
+		(diameter 0)
+		(color 0 0 0 0)
+	)
+	(junction
 		(at 62.23 177.8)
 		(diameter 0)
@@
 					(unit 1)
 				)
+			)
+		)
+	)
+	(symbol
+		(lib_id "power:PWR_FLAG")
+		(at 229.87 86.36 0)
+		(unit 1)
+		(exclude_from_sim no)
+		(in_bom yes)
+		(on_board yes)
+		(dnp no)
+		(fields_autoplaced yes)
+		(property "Reference" "#FLG06"
+			(at 229.87 84.455 0)
+			(effects
+				(font
+					(size 1.27 1.27)
+				)
+				(hide yes)
+			)
+		)
+		(property "Value" "PWR_FLAG"
+			(at 229.87 81.28 0)
+			(effects
+				(font
+					(size 1.27 1.27)
+				)
+			)
+		)
+		(property "Footprint" ""
+			(at 229.87 86.36 0)
+			(effects
+				(font
+					(size 1.27 1.27)
+				)
+				(hide yes)
+			)
+		)
+		(property "Datasheet" "~"
+			(at 229.87 86.36 0)
+			(effects
+				(font
+					(size 1.27 1.27)
+				)
+				(hide yes)
+			)
+		)
+		(property "Description" "Special symbol for telling ERC where power comes from"
+			(at 229.87 86.36 0)
+			(effects
+				(font
+					(size 1.27 1.27)
+				)
+				(hide yes)
+			)
+		)
+		(pin "1"
+		)
+		(instances
+			(project "effectiveRangeHat_simple"
+				(path "/6edc5e63-ec2a-49cc-8eeb-48e0d5e90dc6/a4d8a3cd-2faa-43b2-a96a-f66e8868c6c1"
+					(reference "#FLG06")
+					(unit 1)
+				)

Commit message: fix: pcb changes, moved i2c ext header to 2x2 pin at the edge, pinout adjustments, silkscreen fixes
Parts:
- R34: value 976 -> 1k; MPN ERJ-2RKF9760X -> ERJ-2RKF1001X; SupplierLink https://digikey.hu/en/products/detail/panasonic-electronic-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 -> https://www.digikey.hu/en/products/detail/panasonic-electro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
Changed lines of the file:
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@@
 			)
 		)
-		(property "Value" "976"
+		(property "Value" "1k"
 			(at 222.25 82.55 90)
 			(effects
@@
 			)
 		)
-		(property "MPN" "ERJ-2RKF9760X"
+		(property "MPN" "ERJ-2RKF1001X"
 			(at 222.25 86.36 0)
 			(effects
@@
 			)
 		)
-		(property "SupplierLink" "https://digikey.hu/en/products/detail/panasonic-electronic-components/ERJ-2RKF9760X/192522?s=N4IgjCBcoExaBjKAzAhgGwM4FMA0IB7KAbXABYAGANjJAF18AHAFyhAGVmAnASwDsA5iAC%2B%2BAMzwQSSGix5CJcGDEQGIFm069BI-GCqTpsnPiKRSYgJxgArAA56TVpA7d%2BQ0eADstaFJQYJgrmIGRgYD5wahouWu66IDAUdjaGAXKmipZeVAAEAPIAFgC2mI7qziAAqnw8zPnIALLYqJgArlzYCQC0vojpQWakdnZUlhT0nt0QfkaB8kPgE3TCq0A"
+		(property "SupplierLink" "https://www.digikey.hu/en/products/detail/panasonic-electronic-components/ERJ-2RKF1001X/79729?s=N4IgjCBcoMxaBjKAzAhgGwM4FMA0IB7KAbXDBggF18AHAFyhAGU6AnASwDsBzEAX3xgATAE4I0EEkhoseQiRAwxAVgDsIaiHqMWHHv3xCADAA5l8SSgw58RSKTAACANYB5ABYBbTBtoNIIACqnOx0rsgAstiomACurNgGIAC04ohWsrYKYEYaAikALBZSMjby9iAmJgBsIrmUfI1AA"
 			(at 222.25 86.36 0)
 			(effects
