File: ChargeEnableLogic.kicad_sch (KiCad schematic)
At the start: 29 parts, among them U3 PIC18F16Q20, U4 RX8130CE, U7 SN74CBTLV3257RSVR, U9 GSF7002DW

Commit message: feat: 3V3 regulator + complete rework to 16 layers
Parts:
- removed R29: 1M, Resistor_SMD:R_0402_1005Metric, symbol Device:R
- C13, C29, C36: footprint Capacitor_SMD:C_0805_2012Metric -> Capacitor_SMD:C_0603_1608Metric; MPN GRM21BR61H475KE51L -> GRM188R6YA475KE15D; SupplierLink https://www.digikey.hu/en/products/detail/murata-electronic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 -> https://www.digikey.com/en/products/detail/murata-electroni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
Connections:
- net PIC_ICSPCLK: no longer U3.15 (RA1/ICSPCLK)
- net PIC_ICSPDAT: no longer U3.16 (RA0/ICSPDAT)
- net PIC_RC3 renamed ~{EXT_IRQ}
- net ~{I2C_SEL} renamed PI_5V_DIS
- new net RA0_ICSPDAT: U3.16 (RA0/ICSPDAT)
- new net RA1_ICSPCLK: U3.15 (RA1/ICSPCLK)
Other:
- moved on the sheet: C13, C18, C26, C29, C30, C31, C32, C33, C34, C35, C36, C37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
