File: ft260.kicad_sch (KiCad schematic)
At the start: 15 parts, among them U1 FT230XQ

Commit message: feat: 3V3 regulator + complete rework to 16 layers
Parts:
- C11, C7, C9: footprint Capacitor_SMD:C_0805_2012Metric -> Capacitor_SMD:C_0603_1608Metric; MPN GRM21BR61H475KE51L -> GRM188R6YA475KE15D; SupplierLink https://www.digikey.hu/en/products/detail/murata-electronic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 -> https://www.digikey.com/en/products/detail/murata-electroni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
Changed lines of the file:
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@@
 			)
 		)
-		(property "Footprint" "Capacitor_SMD:C_0805_2012Metric"
+		(property "Footprint" "Capacitor_SMD:C_0603_1608Metric"
 			(at 187.6552 105.41 0)
 			(effects
@@
 			)
 		)
-		(property "MPN" "GRM21BR61H475KE51L"
+		(property "MPN" "GRM188R6YA475KE15D"
 			(at 186.69 101.6 0)
 			(effects
@@
 			)
 		)
-		(property "SupplierLink" "https://www.digikey.hu/en/products/detail/murata-electronics/GRM21BR61H475KE51L/4905540"
+		(property "SupplierLink" "https://www.digikey.com/en/products/detail/murata-electronics/GRM188R6YA475KE15D/3900468"
 			(at 186.69 101.6 0)
 			(effects
@@
 			)
 		)
-		(property "Footprint" "Capacitor_SMD:C_0805_2012Metric"
+		(property "Footprint" "Capacitor_SMD:C_0603_1608Metric"
 			(at 214.3252 81.28 0)
 			(effects
@@
 			)
 		)
-		(property "MPN" "GRM21BR61H475KE51L"
+		(property "MPN" "GRM188R6YA475KE15D"
 			(at 213.36 77.47 0)
 			(effects
@@
 			)
 		)
-		(property "SupplierLink" "https://www.digikey.hu/en/products/detail/murata-electronics/GRM21BR61H475KE51L/4905540"
+		(property "SupplierLink" "https://www.digikey.com/en/products/detail/murata-electronics/GRM188R6YA475KE15D/3900468"
 			(at 213.36 77.47 0)
 			(effects
@@
 			)
 		)
-		(property "Footprint" "Capacitor_SMD:C_0805_2012Metric"
+		(property "Footprint" "Capacitor_SMD:C_0603_1608Metric"
 			(at 187.6552 81.28 0)
 			(effects
@@
 			)
 		)
-		(property "MPN" "GRM21BR61H475KE51L"
+		(property "MPN" "GRM188R6YA475KE15D"
 			(at 186.69 77.47 0)
 			(effects
@@
 			)
 		)
-		(property "SupplierLink" "https://www.digikey.hu/en/products/detail/murata-electronics/GRM21BR61H475KE51L/4905540"
+		(property "SupplierLink" "https://www.digikey.com/en/products/detail/murata-electronics/GRM188R6YA475KE15D/3900468"
 			(at 186.69 77.47 0)
 			(effects
