File: ft260.kicad_sch (KiCad schematic)
At the start: 15 parts, among them U1 FT230XQ

Commit message: v1.14 mods
Parts:
- D2: footprint Diode_SMD:D_0402_1005Metric -> effectiveRangeHat:D_0402_1005Metric
Changed lines of the file:
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@@
 	(label "VCCIN"
 		(at 213.36 69.85 0)
-		(fields_autoplaced yes)
 		(effects
 			(font
@@
 	(label "VCCIN"
 		(at 226.06 69.85 0)
-		(fields_autoplaced yes)
 		(effects
 			(font
@@
 	(label "DP"
 		(at 44.45 92.71 0)
-		(fields_autoplaced yes)
 		(effects
 			(font
@@
 	(label "VOUT3V3"
 		(at 198.12 95.25 0)
-		(fields_autoplaced yes)
 		(effects
 			(font
@@
 	(label "DM"
 		(at 76.2 85.09 0)
-		(fields_autoplaced yes)
 		(effects
 			(font
@@
 	(label "VCCIO"
 		(at 198.12 69.85 0)
-		(fields_autoplaced yes)
 		(effects
 			(font
@@
 	(label "VCCIO"
 		(at 109.22 107.95 0)
-		(fields_autoplaced yes)
 		(effects
 			(font
@@
 	(label "VOUT3V3"
 		(at 124.46 77.47 180)
-		(fields_autoplaced yes)
 		(effects
 			(font
@@
 	(label "D_FT260+"
 		(at 114.3 87.63 0)
-		(fields_autoplaced yes)
 		(effects
 			(font
@@
 	(label "VCCIN"
 		(at 142.24 66.04 180)
-		(fields_autoplaced yes)
 		(effects
 			(font
@@
 	(label "VCCIN"
 		(at 46.99 85.09 0)
-		(fields_autoplaced yes)
 		(effects
 			(font
@@
 	(label "D_FT260-"
 		(at 114.3 85.09 0)
-		(fields_autoplaced yes)
 		(effects
 			(font
@@
 	(label "DM"
 		(at 44.45 90.17 0)
-		(fields_autoplaced yes)
 		(effects
 			(font
@@
 	(label "~{RESET}"
 		(at 123.19 92.71 180)
-		(fields_autoplaced yes)
 		(effects
 			(font
@@
 	(label "VCCIO"
 		(at 147.32 68.58 0)
-		(fields_autoplaced yes)
 		(effects
 			(font
@@
 	(label "DP"
 		(at 76.2 87.63 0)
-		(fields_autoplaced yes)
 		(effects
 			(font
@@
 	(label "VCCIO"
 		(at 186.69 69.85 0)
-		(fields_autoplaced yes)
 		(effects
 			(font
@@
 	(label "~{RESET}"
 		(at 118.11 124.46 0)
-		(fields_autoplaced yes)
 		(effects
 			(font
@@
 	(label "VOUT3V3"
 		(at 186.69 95.25 0)
-		(fields_autoplaced yes)
 		(effects
 			(font
@@
 		(shape input)
 		(at 40.64 90.17 180)
-		(fields_autoplaced yes)
 		(effects
 			(font
@@
 		(shape input)
 		(at 40.64 85.09 180)
-		(fields_autoplaced yes)
 		(effects
 			(font
@@
 		(shape input)
 		(at 40.64 92.71 180)
-		(fields_autoplaced yes)
 		(effects
 			(font
@@
 		(shape output)
 		(at 166.37 80.01 0)
-		(fields_autoplaced yes)
 		(effects
 			(font
@@
 		(shape output)
 		(at 166.37 77.47 0)
-		(fields_autoplaced yes)
 		(effects
 			(font
@@
 			)
 		)
-		(property "Footprint" "Diode_SMD:D_0402_1005Metric"
+		(property "Footprint" "effectiveRangeHat:D_0402_1005Metric"
 			(at 48.26 97.79 0)
 			(effects
