File: effectiveRangeHat_simple.kicad_sch (KiCad schematic)
At the start: 10 parts, among them J1 Raspberry_Pi_2_3, J8 VBUS_EXT, J9 GND_EXT, P1 USB4105GFA120

Commit message: v1.14 mods
Parts:
- removed J8: VBUS_EXT, Connector_PinHeader_2.54mm:PinHeader_1x01_P2.54mm_Vertical, symbol Connector:Conn_01x01_Socket
- removed J9: GND_EXT, Connector_PinHeader_2.54mm:PinHeader_1x01_P2.54mm_Vertical, symbol Connector:Conn_01x01_Socket
- added J8: VBUS_EXT, effectiveRangeHat:CONN02_533750210_MOL, symbol Connector_Generic:Conn_01x02
Connections:
- net GND: now also J8.2 (Pin_2)
- net VBUS: now also J8.1 (Pin_1)
Other:
- sheet Peripheries ports: added ~{MCLR_PI}; removed none

Commit message: connector reorg, trace adjustments
Parts:
- J8: MPN (none) -> 533750210; Manufacturer (none) -> Molex; SupplierLink (none) -> https://www.digikey.hu/en/products/detail/molex/0533750210/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
Changed lines of the file:
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@@
+			)
+		)
+		(property "MPN" "533750210"
+			(at 92.71 31.75 0)
+			(effects
+				(font
+					(size 1.27 1.27)
+				)
+				(hide yes)
+			)
+		)
+		(property "Manufacturer" "Molex"
+			(at 92.71 31.75 0)
+			(effects
+				(font
+					(size 1.27 1.27)
+				)
+				(hide yes)
+			)
+		)
+		(property "SupplierLink" "https://www.digikey.hu/en/products/detail/molex/0533750210/2405348"
+			(at 92.71 31.75 0)
+			(effects
+				(font
+					(size 1.27 1.27)
+				)
+				(hide yes)
 			)
 		)
