File: peri.kicad_sch (KiCad schematic)
At the start: 19 parts, among them J10 EXT_I2S, J4 EXT_BUS, J5 PeriHDR, J6 PI Mating connector, J7 PIC_GPIO, Q1 CSD13381F4, SW4 RP8100B2M1CEBLKBLKWHT, U11 GSF7002DW

Commit message: v1.14 mods
Parts:
- J6: MPN PPPC202LFBN-RC -> 61304021821; Manufacturer Sullins Connector Solutions -> Würth Elektronik
- Q1: footprint Package_TO_SOT_SMD:SOT-883 -> Package_TO_SOT_SMD:SOT-723
Connections:
- net GND: no longer J4.6 (Pin_6)
- new net ~{MCLR_PI}: J4.6 (Pin_6)
Changed lines of the file:
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@@
 	)
 	(junction
-		(at 77.47 63.5)
+		(at 80.01 95.25)
 		(diameter 0)
 		(color 0 0 0 0)
 	)
 	(junction
-		(at 80.01 95.25)
+		(at 229.87 113.03)
 		(diameter 0)
 		(color 0 0 0 0)
 	)
 	(junction
-		(at 229.87 113.03)
+		(at 81.28 63.5)
 		(diameter 0)
 		(color 0 0 0 0)
@@
 	)
 	(junction
-		(at 77.47 60.96)
-		(diameter 0)
-		(color 0 0 0 0)
-	)
-	(junction
 		(at 80.01 90.17)
 		(diameter 0)
@@
 	(wire
 		(pts
-			(xy 68.58 60.96) (xy 77.47 60.96)
-		)
-		(stroke
-			(width 0)
-			(type default)
-		)
-	)
-	(wire
-		(pts
 			(xy 97.79 33.02) (xy 97.79 27.94)
 		)
@@
 	(wire
 		(pts
+			(xy 81.28 63.5) (xy 81.28 71.12)
+		)
+		(stroke
+			(width 0)
+			(type default)
+		)
+	)
+	(wire
+		(pts
 			(xy 140.97 27.94) (xy 140.97 26.67)
 		)
@@
 	(wire
 		(pts
-			(xy 68.58 63.5) (xy 77.47 63.5)
-		)
-		(stroke
-			(width 0)
-			(type default)
-		)
-	)
-	(wire
-		(pts
 			(xy 223.52 60.96) (xy 217.17 60.96)
 		)
@@
 	(wire
 		(pts
-			(xy 77.47 60.96) (xy 77.47 58.42)
+			(xy 81.28 58.42) (xy 81.28 63.5)
 		)
 		(stroke
@@
 	(wire
 		(pts
+			(xy 68.58 63.5) (xy 81.28 63.5)
+		)
+		(stroke
+			(width 0)
+			(type default)
+		)
+	)
+	(wire
+		(pts
 			(xy 73.66 95.25) (xy 80.01 95.25)
 		)
@@
 	(wire
 		(pts
-			(xy 77.47 63.5) (xy 77.47 60.96)
-		)
-		(stroke
-			(width 0)
-			(type default)
-		)
-	)
-	(wire
-		(pts
 			(xy 93.98 91.44) (xy 114.3 91.44)
 		)
@@
 	(wire
 		(pts
-			(xy 77.47 58.42) (xy 68.58 58.42)
-		)
-		(stroke
-			(width 0)
-			(type default)
-		)
-	)
-	(wire
-		(pts
 			(xy 73.66 90.17) (xy 80.01 90.17)
 		)
@@
 	(wire
 		(pts
-			(xy 71.12 66.04) (xy 68.58 66.04)
-		)
-		(stroke
-			(width 0)
-			(type default)
-		)
-	)
-	(wire
-		(pts
 			(xy 80.01 87.63) (xy 80.01 90.17)
 		)
@@
 		)
 	)
-	(wire
-		(pts
-			(xy 77.47 66.04) (xy 77.47 63.5)
-		)
-		(stroke
-			(width 0)
-			(type default)
-		)
-	)
 	(bus
 		(pts
@@
 		)
 	)
+	(wire
+		(pts
+			(xy 68.58 58.42) (xy 81.28 58.42)
+		)
+		(stroke
+			(width 0)
+			(type default)
+		)
+	)
 	(rectangle
 		(start 15.24 17.78)
@@
 	(label "SPI_EXT.MOSI"
 		(at 129.54 86.36 0)
-		(fields_autoplaced yes)
 		(effects
 			(font
@@
 	(label "SPI_EXT.CE0"
 		(at 129.54 93.98 0)
-		(fields_autoplaced yes)
 		(effects
 			(font
@@
 	(label "SPI_EXT.SCLK"
 		(at 129.54 91.44 0)
-		(fields_autoplaced yes)
 		(effects
 			(font
@@
 	(label "ICSP_EXT.CLK"
 		(at 96.52 93.98 0)
-		(fields_autoplaced yes)
 		(effects
 			(font
@@
 	(label "MIC_DOUT"
 		(at 50.8 90.17 0)
-		(fields_autoplaced yes)
 		(effects
 			(font
@@
 	(label "I2S_DIN"
 		(at 58.42 87.63 180)
-		(fields_autoplaced yes)
 		(effects
 			(font
@@
 	(label "ICSP_EXT.DAT"
 		(at 96.52 91.44 0)
-		(fields_autoplaced yes)
 		(effects
 			(font
@@
 	(label "BUZZ_N"
 		(at 229.87 123.19 0)
-		(fields_autoplaced yes)
 		(effects
 			(font
@@
 	(label "Q_BASE"
 		(at 220.98 129.54 180)
-		(fields_autoplaced yes)
 		(effects
 			(font
@@
 	(label "MIC_FS"
 		(at 57.15 82.55 180)
-		(fields_autoplaced yes)
 		(effects
 			(font
@@
 	(label "SPI_EXT.MISO"
 		(at 129.54 88.9 0)
-		(fields_autoplaced yes)
 		(effects
 			(font
@@
 	(label "SPI_EXT.CE1"
 		(at 129.54 96.52 0)
-		(fields_autoplaced yes)
 		(effects
 			(font
@@
 	(label "ICSP_EXT.VDD"
 		(at 96.52 86.36 0)
-		(fields_autoplaced yes)
 		(effects
 			(font
@@
 	(label "ICSP_EXT.~{MCLR}"
 		(at 96.52 83.82 0)
-		(fields_autoplaced yes)
 		(effects
 			(font
@@
 	(label "MIC_CLK"
 		(at 58.42 85.09 180)
-		(fields_autoplaced yes)
 		(effects
 			(font
@@
 		(shape input)
 		(at 34.29 82.55 180)
-		(fields_autoplaced yes)
 		(effects
 			(font
@@
 		(shape input)
 		(at 191.77 129.54 180)
-		(fields_autoplaced yes)
 		(effects
 			(font
@@
 		(shape bidirectional)
 		(at 115.57 40.64 180)
-		(fields_autoplaced yes)
 		(effects
 			(font
@@
 		(shape input)
 		(at 231.14 60.96 0)
-		(fields_autoplaced yes)
 		(effects
 			(font
@@
 		(shape input)
 		(at 185.42 60.96 180)
-		(fields_autoplaced yes)
 		(effects
 			(font
@@
 		(shape output)
 		(at 222.25 57.15 0)
-		(fields_autoplaced yes)
 		(effects
 			(font
@@
 		(shape passive)
 		(at 104.14 66.04 0)
-		(fields_autoplaced yes)
 		(effects
 			(font
@@
 		(shape input)
 		(at 34.29 85.09 180)
-		(fields_autoplaced yes)
 		(effects
 			(font
@@
 		(shape input)
 		(at 189.23 57.15 180)
-		(fields_autoplaced yes)
 		(effects
 			(font
@@
 	(hierarchical_label "GP5"
 		(shape input)
-		(at 71.12 66.04 0)
-		(fields_autoplaced yes)
+		(at 68.58 66.04 0)
 		(effects
 			(font
@@
 		(shape bidirectional)
 		(at 115.57 45.72 180)
-		(fields_autoplaced yes)
 		(effects
 			(font
@@
 		(shape output)
 		(at 35.56 58.42 180)
-		(fields_autoplaced yes)
 		(effects
 			(font
@@
 		(shape input)
 		(at 34.29 95.25 180)
-		(fields_autoplaced yes)
 		(effects
 			(font
@@
 		(shape bidirectional)
 		(at 115.57 30.48 180)
-		(fields_autoplaced yes)
 		(effects
 			(font
@@
 		)
 	)
+	(hierarchical_label "~{MCLR_PI}"
+		(shape input)
+		(at 68.58 60.96 0)
+		(effects
+			(font
+				(size 1.27 1.27)
+			)
+			(justify left)
+		)
+	)
 	(hierarchical_label "SPI_EXT{MOSI MISO SCLK CE0 CE1}"
 		(shape bidirectional)
 		(at 137.16 57.15 180)
-		(fields_autoplaced yes)
 		(effects
 			(font
@@
 		(shape input)
 		(at 54.61 66.04 180)
-		(fields_autoplaced yes)
 		(effects
 			(font
@@
 		(shape output)
 		(at 35.56 63.5 180)
-		(fields_autoplaced yes)
 		(effects
 			(font
@@
 		(shape bidirectional)
 		(at 35.56 60.96 180)
-		(fields_autoplaced yes)
 		(effects
 			(font
@@
 		(shape bidirectional)
 		(at 115.57 35.56 180)
-		(fields_autoplaced yes)
 		(effects
 			(font
@@
 		(shape input)
 		(at 34.29 87.63 180)
-		(fields_autoplaced yes)
 		(effects
 			(font
@@
 		(shape input)
 		(at 34.29 97.79 180)
-		(fields_autoplaced yes)
 		(effects
 			(font
@@
 		(shape input)
 		(at 34.29 90.17 180)
-		(fields_autoplaced yes)
 		(effects
 			(font
@@
 			)
 		)
-		(property "Footprint" "Package_TO_SOT_SMD:SOT-883"
+		(property "Footprint" "Package_TO_SOT_SMD:SOT-723"
 			(at 232.41 131.445 0)
 			(effects
@@
 			)
 		)
-		(property "MPN" "PPPC202LFBN-RC"
+		(property "MPN" "61304021821"
 			(at 45.72 168.91 0)
 			(effects
@@
 			)
 		)
-		(property "Manufacturer" "Sullins Connector Solutions"
+		(property "Manufacturer" "Würth Elektronik"
 			(at 45.72 168.91 0)
 			(effects
@@
 	(symbol
 		(lib_id "power:GND")
-		(at 77.47 66.04 0)
+		(at 81.28 71.12 0)
 		(unit 1)
 		(exclude_from_sim no)
@@
 		(dnp no)
 		(property "Reference" "#PWR079"
-			(at 77.47 72.39 0)
+			(at 81.28 77.47 0)
 			(effects
 				(font
@@
 		)
 		(property "Value" "GND"
-			(at 77.47 71.755 0)
+			(at 81.28 76.835 0)
 			(effects
 				(font
@@
 		)
 		(property "Footprint" ""
-			(at 77.47 66.04 0)
+			(at 81.28 71.12 0)
 			(effects
 				(font
@@
 		)
 		(property "Datasheet" ""
-			(at 77.47 66.04 0)
+			(at 81.28 71.12 0)
 			(effects
 				(font
@@
 		)
 		(property "Description" "Power symbol creates a global label with name \"GND\" , ground"
-			(at 77.47 66.04 0)
+			(at 81.28 71.12 0)
 			(effects
 				(font

Commit message: connector reorg, trace adjustments
Parts:
- removed R40: 33, Resistor_SMD:R_0402_1005Metric, symbol Device:R
- removed TH2: NTCLE213E3103JLB0, symbol Device:Thermistor
- added J9: IO Switch conn., symbol Connector_Generic:Conn_02x02_Odd_Even
- Q1: value CSD13381F4 -> GSFF3134; MPN CSD13381F4 -> GSFF3134; Manufacturer Texas Instruments -> Good-Ark Semiconductor; SupplierLink https://www.digikey.hu/en/products/detail/onsemi/2n7002/244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 -> https://www.digikey.hu/en/products/detail/good-ark-semicond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
- R17: value 33 -> Ext. Pwr Cable; footprint Resistor_SMD:R_0402_1005Metric -> (none); MPN ERJ-2RKF33R0X -> 0151370201; Manufacturer Panasonic Electronic Components -> Molex; SupplierLink https://www.digikey.hu/en/products/detail/panasonic-electro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 -> https://www.digikey.hu/en/products/detail/molex/0151370201/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
- R7: value 33 -> Battery Cable; footprint Resistor_SMD:R_0402_1005Metric -> (none); MPN ERJ-2RKF33R0X -> 0151370301; Manufacturer Panasonic Electronic Components -> Molex; SupplierLink https://www.digikey.hu/en/products/detail/panasonic-electro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 -> https://www.digikey.hu/en/products/detail/molex/0151370301/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
- SW4: MPN RP8100B2M1CEBLKBLKWHT -> PB6B2FM2M1CAL01; Manufacturer E-Switch -> TE Connectivity ALCOSWITCH Switches; SupplierLink https://www.digikey.com/en/products/detail/e-switch/RP8100B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 -> https://www.digikey.hu/en/products/detail/te-connectivity-a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
Connections:
- net MIC_DOUT is gone; now on net I2S_DOUT: J10.9 (Pin_9)
- net I2S_CLK: now also J10.5 (Pin_5); no longer R7.1
- net I2S_FS: now also J10.3 (Pin_3); no longer R17.2
- net MIC_CLK: no longer names the net of R7.2
- net MIC_CLK: no longer J10.5 (Pin_5)
- net MIC_FS: no longer names the net of R17.1
- net MIC_FS: no longer J10.3 (Pin_3)
- no-connect marks 44 -> 50
